Commit message: teleop_keyboard+ultrasonic working

File: urdf/materials.xacro (robot description, xacro)
@@ -1,6 +1,9 @@
 <?xml version="1.0" ?>
 <robot name="rnnbot" xmlns:xacro="http://www.ros.org/wiki/xacro" >
-<material name="silver">
-  <color rgba="0.700 0.700 0.700 1.000"/>
+<material name="black">
+  <color rgba="0.0 0.0 0.0 1.000"/>
+</material>
+<material name="yellow">
+  <color rgba="1.0 1.0 0.0 1.000"/>
 </material>
 </robot>

File: urdf/rnnbot.xacro (robot description, xacro)
@@ -4,4 +4,5 @@
 <xacro:include filename="$(find rnnbot_description)/urdf/rnnbot.trans" />
 <xacro:include filename="$(find rnnbot_description)/urdf/rnnbot.gazebo" />
+<xacro:include filename="$(find rnnbot_description)/urdf/gazebo_control.xacro" />
 <link name="base_link">
   <inertial>
@@ -15,5 +16,5 @@
       <mesh filename="file://$(find rnnbot_description)/meshes/base_link.stl" scale="0.001 0.001 0.001"/>
     </geometry>
-    <material name="silver"/>
+    <material name="yellow"/>
   </visual>
   <collision>
@@ -35,5 +36,5 @@
       <mesh filename="file://$(find rnnbot_description)/meshes/lwheel_link_1.stl" scale="0.001 0.001 0.001"/>
     </geometry>
-    <material name="silver"/>
+    <material name="black"/>
   </visual>
   <collision>
@@ -55,5 +56,5 @@
       <mesh filename="file://$(find rnnbot_description)/meshes/rwheel_link_1.stl" scale="0.001 0.001 0.001"/>
     </geometry>
-    <material name="silver"/>
+    <material name="black"/>
   </visual>
   <collision>
@@ -75,5 +76,5 @@
       <mesh filename="file://$(find rnnbot_description)/meshes/rultrasonic_link_1.stl" scale="0.001 0.001 0.001"/>
     </geometry>
-    <material name="silver"/>
+    <material name="black"/>
   </visual>
   <collision>
@@ -95,5 +96,5 @@
       <mesh filename="file://$(find rnnbot_description)/meshes/fultrasonic_link_1.stl" scale="0.001 0.001 0.001"/>
     </geometry>
-    <material name="silver"/>
+    <material name="black"/>
   </visual>
   <collision>
@@ -115,5 +116,5 @@
       <mesh filename="file://$(find rnnbot_description)/meshes/lultrasonic_link_1.stl" scale="0.001 0.001 0.001"/>
     </geometry>
-    <material name="silver"/>
+    <material name="black"/>
   </visual>
   <collision>
@@ -124,4 +125,31 @@
   </collision>
 </link>
+<link name="lultrasonic_ray_frame"/>
+    <!-- 2. The Joint that twists the invisible frame -->
+<joint name="lultrasonic_ray_joint" type="fixed">
+        <parent link="lultrasonic_link_1"/> <!-- Attached to your physical box -->
+        <child link="lultrasonic_ray_frame"/>
+        <!-- Rotate the invisible frame here! -->
+        <!-- Example: Twist 90 degrees to the left (Yaw: 1.57) -->
+        <origin xyz="0 0 0" rpy="0 0 1.57"/>
+</joint>
+<link name="fultrasonic_ray_frame"/>
+    <!-- 2. The Joint that twists the invisible frame -->
+<joint name="fultrasonic_ray_joint" type="fixed">
+        <parent link="fultrasonic_link_1"/> <!-- Attached to your physical box -->
+        <child link="fultrasonic_ray_frame"/>
+        <!-- Rotate the invisible frame here! -->
+        <!-- Example: Twist 90 degrees to the left (Yaw: 1.57) -->
+        <origin xyz="0 0 0" rpy="0 0 0"/>
+</joint>
+<link name="rultrasonic_ray_frame"/>
+    <!-- 2. The Joint that twists the invisible frame -->
+<joint name="rultrasonic_ray_joint" type="fixed">
+        <parent link="rultrasonic_link_1"/> <!-- Attached to your physical box -->
+        <child link="rultrasonic_ray_frame"/>
+        <!-- Rotate the invisible frame here! -->
+        <!-- Example: Twist 90 degrees to the left (Yaw: 1.57) -->
+        <origin xyz="0 0 0" rpy="0 0 -1.57"/>
+</joint>
 <joint name="lw_joint" type="continuous">
   <origin xyz="0.04 0.19 0.025" rpy="0 0 0"/>
@@ -134,7 +162,7 @@
   <parent link="base_link"/>
   <child link="rwheel_link_1"/>
-  <axis xyz="0.0 -1.0 0.0"/>
+  <axis xyz="0.0 1.0 0.0"/>
 </joint>
-<joint name="lultra_joint" type="fixed">
+<joint name="rultra_joint" type="fixed">
   <origin xyz="0.25 0.0 0.025" rpy="0 0 0"/>
   <parent link="base_link"/>
@@ -146,5 +174,5 @@
   <child link="fultrasonic_link_1"/>
 </joint>
-<joint name="rultra_joint" type="fixed">
+<joint name="lultra_joint" type="fixed">
   <origin xyz="0.25 0.15 0.025" rpy="0 0 0"/>
   <parent link="base_link"/>
